Commit message: Add files via upload

File: my_car_description/urdf/my_car.xacro (robot description, xacro)
@@ -2,6 +2,6 @@
 <robot name="my_car" xmlns:xacro="http://www.ros.org/wiki/xacro">
   <!-- 定义参数 -->
-  <xacro:property name="base_length" value="0.4" />
-  <xacro:property name="base_width" value="0.3" />
+  <xacro:property name="base_length" value="0.6" />
+  <xacro:property name="base_width" value="0.4" />
   <xacro:property name="base_height" value="0.2" />
   <xacro:property name="wheel_radius" value="0.08" />
@@ -24,10 +24,53 @@
     </collision>
     <inertial>
-      <mass value="5.0"/>
-      <inertia ixx="0.1" ixy="0.0" ixz="0.0" iyy="0.1" iyz="0.0" izz="0.1"/>
-    </inertial>
-  </link>
-  <!-- 左轮 -->
-  <link name="left_wheel">
+      <mass value="10.0"/>
+      <inertia ixx="0.2" ixy="0.0" ixz="0.0" iyy="0.2" iyz="0.0" izz="0.2"/>
+    </inertial>
+  </link>
+  <!-- ============================ -->
+  <!-- 车轮定义 - 四个轮子 -->
+  <!-- ============================ -->
+  <!-- 左后轮（驱动轮） -->
+  <link name="left_rear_wheel">
+    <visual>
+      <geometry>
+        <cylinder radius="${wheel_radius}" length="${wheel_width}"/>
+      </geometry>
+      <material name="black">
+        <color rgba="0 0 0 1"/>
+      </material>
+    </visual>
+    <collision>
+      <geometry>
+        <cylinder radius="${wheel_radius}" length="${wheel_width}"/>
+      </geometry>
+    </collision>
+    <inertial>
+      <mass value="0.8"/>
+      <inertia ixx="0.001" ixy="0.0" ixz="0.0" iyy="0.001" iyz="0.0" izz="0.001"/>
+    </inertial>
+  </link>
+  <!-- 右后轮（驱动轮） -->
+  <link name="right_rear_wheel">
+    <visual>
+      <geometry>
+        <cylinder radius="${wheel_radius}" length="${wheel_width}"/>
+      </geometry>
+      <material name="black">
+        <color rgba="0 0 0 1"/>
+      </material>
+    </visual>
+    <collision>
+      <geometry>
+        <cylinder radius="${wheel_radius}" length="${wheel_width}"/>
+      </geometry>
+    </collision>
+    <inertial>
+      <mass value="0.8"/>
+      <inertia ixx="0.001" ixy="0.0" ixz="0.0" iyy="0.001" iyz="0.0" izz="0.001"/>
+    </inertial>
+  </link>
+  <!-- 左前轮（从动轮） -->
+  <link name="left_front_wheel">
     <visual>
       <geometry>
@@ -48,6 +91,6 @@
     </inertial>
   </link>
-  <!-- 右轮 -->
-  <link name="right_wheel">
+  <!-- 右前轮（从动轮） -->
+  <link name="right_front_wheel">
     <visual>
       <geometry>
@@ -68,19 +111,50 @@
     </inertial>
   </link>
-  <!-- 前支撑轮 -->
-  <link name="front_caster">
-    <visual>
-      <geometry>
-        <sphere radius="0.03"/>
-      </geometry>
-      <material name="black">
-        <color rgba="0 0 0 1"/>
-      </material>
-    </visual>
-    <collision>
-      <geometry>
-        <sphere radius="0.03"/>
-      </geometry>
-    </collision>
+  <!-- ============================ -->
+  <!-- 车轮关节 -->
+  <!-- ============================ -->
+  <!-- 左后轮关节（驱动轮） -->
+  <joint name="left_rear_wheel_joint" type="continuous">
+    <parent link="base_link"/>
+    <child link="left_rear_wheel"/>
+    <!-- 车头朝向X轴负方向，所以后轮在X轴正方向 -->
+    <origin xyz="${base_length/4} ${base_width/2} -${base_height/2}" rpy="${PI/2} 0 0"/>
+    <axis xyz="0 1 0"/>
+  </joint>
+  <!-- 右后轮关节（驱动轮） -->
+  <joint name="right_rear_wheel_joint" type="continuous">
+    <parent link="base_link"/>
+    <child link="right_rear_wheel"/>
+    <origin xyz="${base_length/4} -${base_width/2} -${base_height/2}" rpy="${PI/2} 0 0"/>
+    <axis xyz="0 1 0"/>
+  </joint>
+  <!-- 左前轮关节（从动轮） -->
+  <joint name="left_front_wheel_joint" type="continuous">
+    <parent link="base_link"/>
+    <child link="left_front_wheel"/>
+    <!-- 前轮在X轴负方向 -->
+    <origin xyz="-${base_length/4} ${base_width/2} -${base_height/2}" rpy="${PI/2} 0 0"/>
+    <axis xyz="0 1 0"/>
+  </joint>
+  <!-- 右前轮关节（从动轮） -->
+  <joint name="right_front_wheel_joint" type="continuous">
+    <parent link="base_link"/>
+    <child link="right_front_wheel"/>
+    <origin xyz="-${base_length/4} -${base_width/2} -${base_height/2}" rpy="${PI/2} 0 0"/>
+    <axis xyz="0 1 0"/>
+  </joint>
+  <!-- ============================ -->
+  <!-- 传感器配置 -->
+  <!-- ============================ -->
+  <!-- 摄像头连杆（在车头-X轴负方向） -->
+  <link name="camera_link">
+    <visual>
+      <geometry>
+        <box size="0.05 0.05 0.05"/>
+      </geometry>
+      <material name="red">
+        <color rgba="1 0 0 1"/>
+      </material>
+    </visual>
     <inertial>
       <mass value="0.1"/>
@@ -88,19 +162,20 @@
     </inertial>
   </link>
-  <!-- 后支撑轮 -->
-  <link name="rear_caster">
-    <visual>
-      <geometry>
-        <sphere radius="0.03"/>
-      </geometry>
-      <material name="black">
-        <color rgba="0 0 0 1"/>
-      </material>
-    </visual>
-    <collision>
-      <geometry>
-        <sphere radius="0.03"/>
-      </geometry>
-    </collision>
+  <joint name="camera_joint" type="fixed">
+    <parent link="base_link"/>
+    <child link="camera_link"/>
+    <!-- 车头位置，X轴负方向 -->
+    <origin xyz="-${base_length/2 + 0.05} 0 0.1" rpy="0 0 0"/>
+  </joint>
+  <!-- 激光雷达连杆（在车底盘中心，避免扫描到车轮） -->
+  <link name="lidar_link">
+    <visual>
+      <geometry>
+        <cylinder radius="0.03" length="0.05"/>
+      </geometry>
+      <material name="green">
+        <color rgba="0 1 0 1"/>
+      </material>
+    </visual>
     <inertial>
       <mass value="0.1"/>
@@ -108,69 +183,9 @@
     </inertial>
   </link>
-  <!-- 左轮关节 -->
-  <joint name="left_wheel_joint" type="continuous">
-    <parent link="base_link"/>
-    <child link="left_wheel"/>
-    <origin xyz="0 ${base_width/2} -${base_height/2}" rpy="${PI/2} 0 0"/>
-    <axis xyz="0 1 0"/>
-  </joint>
-  <!-- 右轮关节 -->
-  <joint name="right_wheel_joint" type="continuous">
-    <parent link="base_link"/>
-    <child link="right_wheel"/>
-    <origin xyz="0 -${base_width/2} -${base_height/2}" rpy="${PI/2} 0 0"/>
-    <axis xyz="0 1 0"/>
-  </joint>
-  <!-- 前支撑轮关节 -->
-  <joint name="front_caster_joint" type="fixed">
-    <parent link="base_link"/>
-    <child link="front_caster"/>
-    <origin xyz="${base_length/2} 0 -${base_height/2 + 0.03}" rpy="0 0 0"/>
-  </joint>
-  <!-- 后支撑轮关节 -->
-  <joint name="rear_caster_joint" type="fixed">
-    <parent link="base_link"/>
-    <child link="rear_caster"/>
-    <origin xyz="-${base_length/2} 0 -${base_height/2 + 0.03}" rpy="0 0 0"/>
-  </joint>
-  <!-- 摄像头连杆 -->
-  <link name="camera_link">
-    <visual>
-      <geometry>
-        <box size="0.05 0.05 0.05"/>
-      </geometry>
-      <material name="red">
-        <color rgba="1 0 0 1"/>
-      </material>
-    </visual>
-    <inertial>
-      <mass value="0.1"/>
-      <inertia ixx="0.0001" ixy="0.0" ixz="0.0" iyy="0.0001" iyz="0.0" izz="0.0001"/>
-    </inertial>
-  </link>
-  <joint name="camera_joint" type="fixed">
-    <parent link="base_link"/>
-    <child link="camera_link"/>
-    <origin xyz="0.15 0 0.1" rpy="0 0 0"/>
-  </joint>
-  <!-- 激光雷达连杆 -->
-  <link name="lidar_link">
-    <visual>
-      <geometry>
-        <cylinder radius="0.03" length="0.05"/>
-      </geometry>
-      <material name="green">
-        <color rgba="0 1 0 1"/>
-      </material>
-    </visual>
-    <inertial>
-      <mass value="0.1"/>
-      <inertia ixx="0.0001" ixy="0.0" ixz="0.0" iyy="0.0001" iyz="0.0" izz="0.0001"/>
-    </inertial>
-  </link>
   <joint name="lidar_joint" type="fixed">
     <parent link="base_link"/>
     <child link="lidar_link"/>
-    <origin xyz="0 0 0.15" rpy="0 0 0"/>
+    <!-- 车底盘中心，提高位置避免扫描到车轮 -->
+    <origin xyz="0 0 -${base_height/2 + 0.1}" rpy="0 0 0"/>
   </joint>
   <!-- ============================ -->
@@ -181,11 +196,17 @@
     <material>Gazebo/Blue</material>
   </gazebo>
-  <gazebo reference="left_wheel">
-    <material>Gazebo/Black</material>
-  </gazebo>
-  <gazebo reference="right_wheel">
-    <material>Gazebo/Black</material>
-  </gazebo>
-  <!-- 差速驱动插件 -->
+  <gazebo reference="left_rear_wheel">
+    <material>Gazebo/Black</material>
+  </gazebo>
+  <gazebo reference="right_rear_wheel">
+    <material>Gazebo/Black</material>
+  </gazebo>
+  <gazebo reference="left_front_wheel">
+    <material>Gazebo/Black</material>
+  </gazebo>
+  <gazebo reference="right_front_wheel">
+    <material>Gazebo/Black</material>
+  </gazebo>
+  <!-- 差速驱动插件（只控制后轮） -->
   <gazebo>
     <plugin name="differential_drive_controller" filename="libgazebo_ros_diff_drive.so">
@@ -197,10 +218,10 @@
       <wheelSeparation>${base_width}</wheelSeparation>
       <wheelDiameter>${2 * wheel_radius}</wheelDiameter>
-      <maxWheelTorque>20</maxWheelTorque>
+      <maxWheelTorque>30</maxWheelTorque>
       <maxWheelAcceleration>1.0</maxWheelAcceleration>
       <publishWheelTF>false</publishWheelTF>
       <publishTf>true</publishTf>
-      <leftJoint>left_wheel_joint</leftJoint>
-      <rightJoint>right_wheel_joint</rightJoint>
+      <leftJoint>left_rear_wheel_joint</leftJoint>
+      <rightJoint>right_rear_wheel_joint</rightJoint>
     </plugin>
   </gazebo>
@@ -237,5 +258,5 @@
     </sensor>
   </gazebo>
-  <!-- 激光雷达插件 -->
+  <!-- 激光雷达插件 - 调整参数避免扫描到车轮 -->
   <gazebo reference="lidar_link">
     <sensor type="ray" name="lidar">
@@ -253,5 +274,5 @@
         </scan>
         <range>
-          <min>0.10</min>
+          <min>0.15</min>  <!-- 增加最小距离避免扫描到车轮 -->
           <max>10.0</max>
           <resolution>0.01</resolution>
